File: hardware/GadgetBox-Photon/Gadget-Box-Photon-modules.brd (EAGLE design)
At the start: 93.5 x 53.5 mm, 15 parts

Commit message: photon IO selected
still need CS for SPI ports
Parts:
- added BAT1: (no value), SparkFun-Electromechanical:BATTCON_12MM
Connections:
- removed net N$10: AL.G7, BH.G0
- removed net N$11: AH.G0, BL.G7
- removed net N$12: AH.G1, BL.G6
- removed net N$13: AH.G2, BL.G5
- removed net N$14: AH.G3, BL.G4
- removed net N$15: AH.G4, BL.G3
- removed net N$16: AH.G5, BL.G2
- removed net N$17: AH.G6, BL.G1
- removed net N$18: AH.G7, BL.G0
- removed net N$4: AL.G1, BH.G6
- removed net N$5: AL.G2, BH.G5
- removed net N$6: AL.G3, BH.G4
- removed net N$7: AL.G4, BH.G3
- removed net N$8: AL.G5, BH.G2
- removed net N$9: AL.G6, BH.G1
- removed net VBAT: U$7.22
- new net GB0: AL.G0, BH.G7, U$7.4
- new net GB1: AL.G1, BH.G6, U$7.3
- new net GB10: AH.G2, BL.G5, U$7.27
- new net GB11: AH.G3, BL.G4, U$7.28
- new net GB12: AH.G4, BL.G3, U$7.29
- new net GB13: AH.G5, BL.G2, U$7.18
- new net GB14: AH.G6, BL.G1, U$7.19
- new net GB15: AH.G7, BL.G0, U$7.20
- new net GB2: AL.G2, BH.G5, U$7.17
- new net GB3: AL.G3, BH.G4, U$7.16
- new net GB4: AL.G4, BH.G3, U$7.15
- new net GB5: AL.G5, BH.G2, U$7.5
- new net GB6: AL.G6, BH.G1, U$7.10
- new net GB7: AL.G7, BH.G0, U$7.6
- new net GB8: AH.G0, BL.G7, U$7.12
- new net GB9: AH.G1, BL.G6, U$7.11
- new net RESET: AH.RESET@B6, AL.RESET@B6, BH.RESET@B6, BL.RESET@B6, U$7.23
- net GND: now also BAT1.GND
- net N$3: now also BAT1.PWR@1, U$7.22; no longer AL.G0, BH.G7
